File: kicad/heaterboard.kicad_pcb (KiCad board)
At the start: 2 copper layers, 68.6 x 53.3 mm, 15 parts, among them J1 Power, J2 Digital/PWM, J3 Analog, J4 Digital/PWM, J5 Screw_Terminal_01x02, J6 Screw_Terminal_01x02, Q1 Q_NMOS_GDS, U1 LM7805_TO220

Commit message: design pass 1
Parts:
- added J7: Conn_01x05_Pin, Connector_PinHeader_2.54mm:PinHeader_1x05_P2.54mm_Vertical, F.Cu at (107.6, 51.7)
- added R3: 15 kΩ, Resistor_THT:R_Axial_DIN0207_L6.3mm_D2.5mm_P10.16mm_Horizontal, F.Cu at (145.7, 74.6)
- added R4: 5 kΩ, Resistor_THT:R_Axial_DIN0207_L6.3mm_D2.5mm_P10.16mm_Horizontal, F.Cu at (145.7, 82.2)
- R1: value R,IEEE -> 10 kΩ
- R2: value R,IEEE -> 5 kΩ
- moved R1 18.0 mm to (145.7, 59.4)
- moved R2 18.0 mm to (145.7, 67.0)
- moved Q1 13.7 mm to (133.0, 74.6)
- moved U1 12.7 mm to (133.0, 59.4)
Connections:
- R1 pad 2: Net-(R1--) -> /A3
- R2 pad 1: Net-(R1--) -> /A3
- TH1 pad 2: unconnected-(TH1-Pad2) -> /A2

Commit message: end of class 30 jan
Connections:
- J1 pad 6: GND -> Net-(J1-Pin_6)
- J1 pad 7: GND -> Net-(J1-Pin_6)
- J2 pad 4: GND -> unconnected-(J2-Pin_4-Pad4)
- J5 pad 1: GND -> unconnected-(J5-Pin_1-Pad1)
- J5 pad 2: VCC -> unconnected-(J5-Pin_2-Pad2)
- U1 pad 2: GND -> Net-(J1-Pin_6)
Routing:
- net unconnected-(J5-Pin_1-Pad1): track 0.00 -> 98.2 mm, vias 0 -> 1
- net /SCL/A5: track 0.00 -> 73.2 mm
- net /SDA/A4: track 0.00 -> 71.1 mm
- net /A2: track 0.00 -> 58.4 mm
- net Net-(J7-Pin_5): track 0.00 -> 56.7 mm
- net /A3: track 0.00 -> 51.5 mm
- net Net-(J7-Pin_3): track 0.00 -> 45.5 mm
- net Net-(J1-Pin_6): track 0.00 -> 45.4 mm, vias 0 -> 1
- net VCC: track 0.00 -> 41.4 mm
- net /*3: track 0.00 -> 34.9 mm
- net /A1: track 0.00 -> 31.2 mm
- net Net-(J6-Pin_1): track 0.00 -> 30.0 mm
- net Net-(J7-Pin_2): track 0.00 -> 6.50 mm
