File: kicad/heaterboard.kicad_sch (KiCad schematic)
At the start: 4 parts, among them Q1 PSMN1R0-30YLC_115, U1 LM7805_TO220

Commit message: end of class 25 jan
Parts:
- removed A1: Arduino_UNO_R3, Module:Arduino_UNO_R3, symbol MCU_Module:Arduino_UNO_R3
- removed Q1: PSMN1R0-30YLC_115, PSMN1R0-30YLC_115:DPAK127P_600X120-5N, symbol PSMN1R0-30YLC_115:PSMN1R0-30YLC_115
- added J1: Power, Connector_PinSocket_2.54mm:PinSocket_1x08_P2.54mm_Vertical, symbol Connector_Generic:Conn_01x08
- added J2: Digital/PWM, Connector_PinSocket_2.54mm:PinSocket_1x10_P2.54mm_Vertical, symbol Connector_Generic:Conn_01x10
- added J3: Analog, Connector_PinSocket_2.54mm:PinSocket_1x06_P2.54mm_Vertical, symbol Connector_Generic:Conn_01x06
- added J4: Digital/PWM, Connector_PinSocket_2.54mm:PinSocket_1x08_P2.54mm_Vertical, symbol Connector_Generic:Conn_01x08
- added J5, J6: Screw_Terminal_01x02, Connector_PinHeader_2.54mm:PinHeader_1x02_P2.54mm_Vertical, symbol Connector:Screw_Terminal_01x02
- added Q1: Q_NMOS_GDS, Package_TO_SOT_THT:TO-220-3_Vertical, symbol Device:Q_NMOS_GDS
- added R1: 10 kΩ, Resistor_THT:R_Axial_DIN0207_L6.3mm_D2.5mm_P10.16mm_Horizontal, symbol PCM_Generic:R,IEEE
- added R2: 5 kΩ, Resistor_THT:R_Axial_DIN0207_L6.3mm_D2.5mm_P10.16mm_Horizontal, symbol PCM_Generic:R,IEEE
- TH1: footprint (none) -> Connector_JST:JST_XH_B2B-XH-A_1x02_P2.50mm_Vertical
Connections:
- net GND: now reaches U1.2 (GND)
- net GND: now also J1.6 (Pin_6), J1.7 (Pin_7), J2.4 (Pin_4), J5.1 (Pin_1)
- net A0: now reaches TH1.2
- net A0: now also J3.1 (Pin_1)
- new net: J6.1 (Pin_1), Q1.2 (D)
- new net *10: J2.8 (Pin_8)
- new net *11: J2.7 (Pin_7)
- new net *3: J4.5 (Pin_5), Q1.1 (G)
- new net *5: J4.3 (Pin_3)
- new net *9: J2.9 (Pin_9)
- new net +3V3: J1.4 (Pin_4)
- new net +5V: J1.5 (Pin_5)
- new net 12: J2.6 (Pin_6)
- new net 13: J2.5 (Pin_5)
- new net 2: J4.6 (Pin_6)
- new net 4: J4.4 (Pin_4)
- new net 8: J2.10 (Pin_10)
- new net A1: J3.2 (Pin_2), R1.2 (-), R2.1 (+)
- new net A2: J3.3 (Pin_3)
- new net A3: J3.4 (Pin_4)
- new net AREF: J2.3 (Pin_3)
- new net IOREF: J1.2 (Pin_2)
- new net RX/0: J4.8 (Pin_8)
- new net SCL/A5: J2.1 (Pin_1), J3.6 (Pin_6)
- new net SDA/A4: J2.2 (Pin_2), J3.5 (Pin_5)
- new net TX/1: J4.7 (Pin_7)
- new net VCC: J1.8 (Pin_8), J5.2 (Pin_2)
- new net ~{RESET}: J1.3 (Pin_3)
- no-connect marks 0 -> 1
Other:
- note added: "* Indicates a PWM-capable pin"
- company: (none) -> ME692
- title: (none) -> Windhsield Heater Controller

Commit message: design pass 1
Parts:
- added J7: Conn_01x05_Pin, Connector_PinHeader_2.54mm:PinHeader_1x05_P2.54mm_Vertical, symbol Connector:Conn_01x05_Pin
- added R3: 15 kΩ, Resistor_THT:R_Axial_DIN0207_L6.3mm_D2.5mm_P10.16mm_Horizontal, symbol PCM_Generic:R,IEEE
- added R4: 5 kΩ, Resistor_THT:R_Axial_DIN0207_L6.3mm_D2.5mm_P10.16mm_Horizontal, symbol PCM_Generic:R,IEEE
Connections:
- net A0: no longer TH1.2
- net A1: now also R3.2 (-), R4.1 (+); no longer R1.2 (-), R2.1 (+)
- net A2: now also TH1.2
- net A3: now also R1.2 (-), R2.1 (+)
- new net: J7.3 (Pin_3), R3.1 (+)
- new net: J7.2 (Pin_2), J7.4 (Pin_4)
- new net: J7.5 (Pin_5), R4.2 (-)
Other:
- note added: "RF control module link"
Changed lines of the file:
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@@
     (company "ME692")
   )
+  (junction (at 203.2 127) (diameter 0) (color 0 0 0 0)
+  )
   (junction (at 31.75 46.99) (diameter 1.016) (color 0 0 0 0)
   )
+  (junction (at 203.2 67.31) (diameter 0) (color 0 0 0 0)
+  )
   (junction (at 152.4 76.2) (diameter 0) (color 0 0 0 0)
+  )
+  (junction (at 190.5 113.03) (diameter 0) (color 0 0 0 0)
   )
   (no_connect (at 34.29 31.75))
@@
     (stroke (width 0) (type default))
   )
+  (bus_entry (at 200.66 25.4) (size 2.54 2.54)
+    (stroke (width 0) (type default))
+  )
   (bus_entry (at 101.6 50.8) (size 2.54 -2.54)
     (stroke (width 0) (type default))
@@
     (stroke (width 0) (type default))
   )
+  (bus_entry (at 200.66 152.4) (size 2.54 -2.54)
+    (stroke (width 0) (type default))
+  )
   (wire (pts (xy 62.23 77.47) (xy 74.93 77.47))
     (stroke (width 0) (type solid))
@@
     (stroke (width 0) (type solid))
   )
+  (wire (pts (xy 19.05 87.63) (xy 19.05 67.31))
+    (stroke (width 0) (type default))
+  )
   (bus (pts (xy 124.46 152.4) (xy 149.86 152.4))
     (stroke (width 0) (type default))
@@
     (stroke (width 0) (type default))
   )
+  (wire (pts (xy 21.59 59.69) (xy 34.29 59.69))
+    (stroke (width 0) (type default))
+  )
   (wire (pts (xy 29.21 41.91) (xy 34.29 41.91))
     (stroke (width 0) (type solid))
@@
     (stroke (width 0) (type solid))
   )
+  (wire (pts (xy 13.97 62.23) (xy 34.29 62.23))
+    (stroke (width 0) (type default))
+  )
   (wire (pts (xy 152.4 27.94) (xy 152.4 63.5))
     (stroke (width 0) (type default))
@@
     (stroke (width 0) (type default))
   )
-  (wire (pts (xy 16.51 59.69) (xy 34.29 59.69))
-    (stroke (width 0) (type solid))
-  )
   (wire (pts (xy 62.23 39.37) (xy 74.93 39.37))
     (stroke (width 0) (type solid))
   )
+  (wire (pts (xy 190.5 113.03) (xy 190.5 114.3))
+    (stroke (width 0) (type default))
+  )
   (bus (pts (xy 175.26 25.4) (xy 149.86 25.4))
     (stroke (width 0) (type default))
   )
-  (wire (pts (xy 16.51 90.17) (xy 16.51 59.69))
+  (wire (pts (xy 16.51 90.17) (xy 16.51 64.77))
     (stroke (width 0) (type default))
   )
@@
     (stroke (width 0) (type solid))
   )
+  (wire (pts (xy 203.2 149.86) (xy 203.2 127))
+    (stroke (width 0) (type default))
+  )
   (wire (pts (xy 139.7 87.63) (xy 139.7 76.2))
     (stroke (width 0) (type default))
   )
-  (wire (pts (xy 34.29 64.77) (xy 21.59 64.77))
-    (stroke (width 0) (type solid))
+  (bus (pts (xy 200.66 25.4) (xy 254 25.4))
+    (stroke (width 0) (type default))
   )
   (wire (pts (xy 19.05 36.83) (xy 34.29 36.83))
     (stroke (width 0) (type solid))
   )
+  (bus (pts (xy 200.66 152.4) (xy 266.7 152.4))
+    (stroke (width 0) (type default))
+  )
   (wire (pts (xy 34.29 46.99) (xy 31.75 46.99))
     (stroke (width 0) (type solid))
@@
     (stroke (width 0) (type default))
   )
+  (wire (pts (xy 190.5 124.46) (xy 190.5 127))
+    (stroke (width 0) (type default))
+  )
   (bus (pts (xy 88.9 50.8) (xy 101.6 50.8))
     (stroke (width 0) (type default))
@@
     (stroke (width 0) (type solid))
   )
-  (wire (pts (xy 19.05 62.23) (xy 34.29 62.23))
-    (stroke (width 0) (type solid))
+  (wire (pts (xy 190.5 127) (xy 203.2 127))
+    (stroke (width 0) (type default))
   )
   (wire (pts (xy 139.7 76.2) (xy 152.4 76.2))
     (stroke (width 0) (type default))
   )
+  (wire (pts (xy 190.5 69.85) (xy 205.74 69.85))
+    (stroke (width 0) (type default))
+  )
+  (wire (pts (xy 203.2 72.39) (xy 203.2 67.31))
+    (stroke (width 0) (type default))
+  )
   (wire (pts (xy 62.23 34.29) (xy 64.77 34.29))
     (stroke (width 0) (type solid))
   )
+  (wire (pts (xy 16.51 64.77) (xy 34.29 64.77))
+    (stroke (width 0) (type solid))
+  )
   (bus (pts (xy 124.46 25.4) (xy 149.86 25.4))
     (stroke (width 0) (type default))
@@
     (stroke (width 0) (type solid))
   )
+  (wire (pts (xy 190.5 113.03) (xy 13.97 113.03))
+    (stroke (width 0) (type default))
+  )
   (wire (pts (xy 62.23 41.91) (xy 74.93 41.91))
     (stroke (width 0) (type solid))
   )
-  (bus (pts (xy 175.26 25.4) (xy 254 25.4))
+  (wire (pts (xy 203.2 67.31) (xy 203.2 27.94))
+    (stroke (width 0) (type default))
+  )
+  (wire (pts (xy 203.2 74.93) (xy 205.74 74.93))
+    (stroke (width 0) (type default))
+  )
+  (bus (pts (xy 175.26 25.4) (xy 200.66 25.4))
     (stroke (width 0) (type default))
   )
@@
     (stroke (width 0) (type default))
   )
-  (bus (pts (xy 149.86 152.4) (xy 266.7 152.4))
+  (bus (pts (xy 149.86 152.4) (xy 200.66 152.4))
     (stroke (width 0) (type default))
   )
@@
     (stroke (width 0) (type solid))
   )
-  (wire (pts (xy 21.59 67.31) (xy 34.29 67.31))
+  (wire (pts (xy 203.2 127) (xy 203.2 74.93))
+    (stroke (width 0) (type default))
+  )
+  (wire (pts (xy 19.05 67.31) (xy 34.29 67.31))
     (stroke (width 0) (type solid))
   )
@@
     (stroke (width 0) (type default))
   )
+  (wire (pts (xy 205.74 72.39) (xy 203.2 72.39))
+    (stroke (width 0) (type default))
+  )
   (wire (pts (xy 177.8 90.17) (xy 177.8 73.66))
     (stroke (width 0) (type default))
   )
+  (wire (pts (xy 13.97 113.03) (xy 13.97 62.23))
+    (stroke (width 0) (type default))
+  )
   (wire (pts (xy 62.23 29.21) (xy 74.93 29.21))
     (stroke (width 0) (type solid))
@@
     (stroke (width 0) (type solid))
   )
+  (wire (pts (xy 190.5 111.76) (xy 190.5 113.03))
+    (stroke (width 0) (type default))
+  )
   (wire (pts (xy 62.23 74.93) (xy 74.93 74.93))
     (stroke (width 0) (type solid))
@@
     (stroke (width 0) (type solid))
   )
+  (wire (pts (xy 190.5 101.6) (xy 190.5 69.85))
+    (stroke (width 0) (type default))
+  )
+  (wire (pts (xy 203.2 67.31) (xy 205.74 67.31))
+    (stroke (width 0) (type default))
+  )
   (wire (pts (xy 34.29 69.85) (xy 21.59 69.85))
     (stroke (width 0) (type solid))
@@
     (stroke (width 0) (type solid))
   )
-  (wire (pts (xy 19.05 87.63) (xy 19.05 62.23))
-    (stroke (width 0) (type default))
-  )
   (bus (pts (xy 101.6 50.8) (xy 254 50.8))
     (stroke (width 0) (type default))
+  )
+  (text "RF control module link" (at 205.74 77.47 0)
+    (effects (font (size 1.27 1.27)) (justify left bottom) (href "https://www.amazon.com/DieseRC-Universal-Wireless-Receiver-Transmitters/dp/B098X9GFGB"))
   )
   (text "* Indicates a PWM-capable pin" (at 38.1 82.55 0)
@@
     )
   )
+  (symbol (lib_id "PCM_Generic:R,IEEE") (at 190.5 106.68 0) (unit 1)
+    (in_bom yes) (on_board yes) (dnp no) (fields_autoplaced)
+    (property "Reference" "R3" (at 193.04 104.1399 0)
+      (effects (font (size 2.54 2.54)) (justify left))
+    )
+    (property "Value" "15 kΩ" (at 193.04 109.2199 0)
+      (effects (font (size 2.54 2.54)) (justify left))
+    )
+    (property "Footprint" "Resistor_THT:R_Axial_DIN0207_L6.3mm_D2.5mm_P10.16mm_Horizontal" (at 190.5 106.68 0)
+      (effects (font (size 2.54 2.54)) hide)
+    )
+    (property "Datasheet" "" (at 190.5 106.68 0)
+      (effects (font (size 2.54 2.54)) hide)
+    )
+    (property "Indicator" "+" (at 187.96 104.14 0)
+      (effects (font (size 1.27 1.27)) hide)
+    )
+    (pin "1")
+    (pin "2")
+    (instances
+      (project "heaterboard"
+        (path "/e63e39d7-6ac0-4ffd-8aa3-1841a4541b55"
+          (reference "R3") (unit 1)
+        )
+      )
+    )
+  )
   (symbol (lib_id "Connector:Screw_Terminal_01x02") (at 26.67 134.62 180) (unit 1)
     (in_bom yes) (on_board yes) (dnp no) (fields_autoplaced)
@@
     )
   )
+  (symbol (lib_id "Connector:Conn_01x05_Pin") (at 210.82 69.85 0) (mirror y) (unit 1)
+    (in_bom yes) (on_board yes) (dnp no)
+    (property "Reference" "J7" (at 210.185 59.69 0)
+      (effects (font (size 1.27 1.27)))
+    )
+    (property "Value" "Conn_01x05_Pin" (at 210.185 62.23 0)
+      (effects (font (size 1.27 1.27)))
+    )
+    (property "Footprint" "Connector_PinHeader_2.54mm:PinHeader_1x05_P2.54mm_Vertical" (at 210.82 69.85 0)
+      (effects (font (size 1.27 1.27)) hide)
+    )
+    (property "Datasheet" "~" (at 210.82 69.85 0)
+      (effects (font (size 1.27 1.27)) hide)
+    )
+    (pin "4")
+    (pin "2")
+    (pin "3")
+    (pin "5")
+    (pin "1")
+    (instances
+      (project "heaterboard"
+        (path "/e63e39d7-6ac0-4ffd-8aa3-1841a4541b55"
+          (reference "J7") (unit 1)
+        )
+      )
+    )
+  )
   (symbol (lib_id "PCM_Generic:R,IEEE") (at 152.4 68.58 0) (unit 1)
     (in_bom yes) (on_board yes) (dnp no) (fields_autoplaced)
@@
         )
       )
+    )
+  )
+  (symbol (lib_id "PCM_Generic:R,IEEE") (at 190.5 119.38 0) (unit 1)
+    (in_bom yes) (on_board yes) (dnp no) (fields_autoplaced)
+    (property "Reference" "R4" (at 193.04 116.8399 0)
+      (effects (font (size 2.54 2.54)) (justify left))
+    )
+    (property "Value" "5 kΩ" (at 193.04 121.9199 0)
+      (effects (font (size 2.54 2.54)) (justify left))
+    )
+    (property "Footprint" "Resistor_THT:R_Axial_DIN0207_L6.3mm_D2.5mm_P10.16mm_Horizontal" (at 190.5 119.38 0)
+      (effects (font (size 2.54 2.54)) hide)
+    )
+    (property "Datasheet" "" (at 190.5 119.38 0)
+      (effects (font (size 2.54 2.54)) hide)
+    )
+    (property "Indicator" "+" (at 187.96 116.84 0)
+      (effects (font (size 1.27 1.27)) hide)
+    )
+    (pin "1")
+    (pin "2")
+    (instances
+      (project "heaterboard"
+        (path "/e63e39d7-6ac0-4ffd-8aa3-1841a4541b55"
+          (reference "R4") (unit 1)
+        )
+      )

Commit message: end of class 30 jan
Connections:
- net GND: no longer J1.6 (Pin_6), J1.7 (Pin_7), J2.4 (Pin_4), J5.1 (Pin_1), U1.2 (GND)
- net VCC: no longer J5.2 (Pin_2)
- new net: J1.6 (Pin_6), J1.7 (Pin_7), U1.2 (GND)
Other:
- moved on the sheet: J5, J6
