File: kicad/V1/heaterboard.kicad_pcb (KiCad board)
At the start: 2 copper layers, 68.6 x 53.3 mm, 18 parts, among them J1 Power, J2 Digital/PWM, J3 Analog, J4 Digital/PWM, J5 Screw_Terminal_01x02, J6 Screw_Terminal_01x02, J7 Conn_01x05_Pin, Q1 Q_NMOS_GDS, U1 LM7805_TO220

Commit message: pivot to nano
Routing:
- net unconnected-(J5-Pin_1-Pad1): track 98.2 -> 0.00 mm, vias 1 -> 0
- net /SCL/A5: track 73.2 -> 0.00 mm
- net /SDA/A4: track 71.1 -> 0.00 mm
- net /A2: track 58.4 -> 0.00 mm
- net Net-(J7-Pin_5): track 56.7 -> 0.00 mm
- net /A3: track 51.5 -> 0.00 mm
- net Net-(J7-Pin_3): track 45.5 -> 0.00 mm
- net Net-(J1-Pin_6): track 45.4 -> 0.00 mm, vias 1 -> 0
- net VCC: track 41.4 -> 0.00 mm
- net /*3: track 34.9 -> 0.00 mm
- net /A1: track 31.2 -> 0.00 mm
- net Net-(J6-Pin_1): track 30.0 -> 0.00 mm
- net Net-(J7-Pin_2): track 6.50 -> 0.00 mm
Other:
- copper layers 2 -> 4
Changed lines of the file:
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@@
   (layers
     (0 "F.Cu" signal)
+    (1 "In1.Cu" signal)
+    (2 "In2.Cu" signal)
     (31 "B.Cu" signal)
     (32 "B.Adhes" user "B.Adhesive")
@@
       (layer "F.Mask" (type "Top Solder Mask") (color "Green") (thickness 0.01))
       (layer "F.Cu" (type "copper") (thickness 0.035))
-      (layer "dielectric 1" (type "core") (thickness 1.51) (material "FR4") (epsilon_r 4.5) (loss_tangent 0.02))
+      (layer "dielectric 1" (type "prepreg") (thickness 0.1) (material "FR4") (epsilon_r 4.5) (loss_tangent 0.02))
+      (layer "In1.Cu" (type "copper") (thickness 0.035))
+      (layer "dielectric 2" (type "core") (thickness 1.24) (material "FR4") (epsilon_r 4.5) (loss_tangent 0.02))
+      (layer "In2.Cu" (type "copper") (thickness 0.035))
+      (layer "dielectric 3" (type "prepreg") (thickness 0.1) (material "FR4") (epsilon_r 4.5) (loss_tangent 0.02))
       (layer "B.Cu" (type "copper") (thickness 0.035))
       (layer "B.Mask" (type "Bottom Solder Mask") (color "Green") (thickness 0.01))
@@
     (effects (font (size 1 1) (thickness 0.15)))
   )
-  (segment (start 138.6203 57.9877) (end 143.6635 63.0309) (width 0.25) (layer "F.Cu") (net 1))
-  (segment (start 143.6635 63.0309) (end 143.6635 64.8556) (width 0.25) (layer "F.Cu") (net 1))
-  (segment (start 136.9323 57.9877) (end 138.6203 57.9877) (width 0.25) (layer "F.Cu") (net 1))
-  (segment (start 135.56 59.36) (end 136.9323 57.9877) (width 0.25) (layer "F.Cu") (net 1))
-  (via (at 143.6635 64.8556) (size 0.6) (drill 0.4) (layers "F.Cu" "B.Cu") (net 1))
-  (segment (start 143.18 65.3391) (end 143.6635 64.8556) (width 0.25) (layer "B.Cu") (net 1))
-  (segment (start 143.18 97.46) (end 143.18 65.3391) (width 0.25) (layer "B.Cu") (net 1))
-  (segment (start 147.757 90.7001) (end 153.34 96.2831) (width 0.25) (layer "B.Cu") (net 6))
-  (segment (start 155.88 74.6) (end 154.753 74.6) (width 0.25) (layer "B.Cu") (net 6))
-  (segment (start 147.757 82.22) (end 145.72 82.22) (width 0.25) (layer "B.Cu") (net 6))
-  (segment (start 147.757 82.22) (end 147.757 90.7001) (width 0.25) (layer "B.Cu") (net 6))
-  (segment (start 153.34 96.2831) (end 153.34 97.46) (width 0.25) (layer "B.Cu") (net 6))
-  (segment (start 147.757 81.596) (end 147.757 82.22) (width 0.25) (layer "B.Cu") (net 6))
-  (segment (start 154.753 74.6) (end 147.757 81.596) (width 0.25) (layer "B.Cu") (net 6))
-  (segment (start 154.703 97.0942) (end 137.329 79.72) (width 0.25) (layer "F.Cu") (net 7))
-  (segment (start 154.703 97.46) (end 154.703 97.0942) (width 0.25) (layer "F.Cu") (net 7))
-  (segment (start 155.88 97.46) (end 154.703 97.46) (width 0.25) (layer "F.Cu") (net 7))
-  (segment (start 137.329 79.72) (end 105.08 79.72) (width 0.25) (layer "F.Cu") (net 7))
-  (segment (start 147.133 66.98) (end 145.72 66.98) (width 0.25) (layer "F.Cu") (net 8))
-  (segment (start 154.753 59.36) (end 147.133 66.98) (width 0.25) (layer "F.Cu") (net 8))
-  (segment (start 155.88 59.36) (end 154.753 59.36) (width 0.25) (layer "F.Cu") (net 8))
-  (segment (start 145.72 66.98) (end 149.882 66.98) (width 0.25) (layer "B.Cu") (net 8))
-  (segment (start 149.882 66.98) (end 158.42 75.5179) (width 0.25) (layer "B.Cu") (net 8))
-  (segment (start 158.42 75.5179) (end 158.42 97.46) (width 0.25) (layer "B.Cu") (net 8))
-  (segment (start 158.948 98.6609) (end 159.783 97.8258) (width 0.25) (layer "F.Cu") (net 9))
-  (segment (start 159.783 97.46) (end 160.96 97.46) (width 0.25) (layer "F.Cu") (net 9))
-  (segment (start 136.425 61.1545) (end 157.15 81.8793) (width 0.25) (layer "F.Cu") (net 9))
-  (segment (start 157.15 81.8793) (end 157.15 97.8807) (width 0.25) (layer "F.Cu") (net 9))
-  (segment (start 121.336 49.2) (end 121.336 50.7753) (width 0.25) (layer "F.Cu") (net 9))
-  (segment (start 157.15 97.8807) (end 157.93 98.6609) (width 0.25) (layer "F.Cu") (net 9))
-  (segment (start 131.715 61.1545) (end 136.425 61.1545) (width 0.25) (layer "F.Cu") (net 9))
-  (segment (start 121.336 50.7753) (end 131.715 61.1545) (width 0.25) (layer "F.Cu") (net 9))
-  (segment (start 159.783 97.8258) (end 159.783 97.46) (width 0.25) (layer "F.Cu") (net 9))
-  (segment (start 157.93 98.6609) (end 158.948 98.6609) (width 0.25) (layer "F.Cu") (net 9))
-  (segment (start 136.614 60.7025) (end 163.5 87.5882) (width 0.25) (layer "F.Cu") (net 10))
-  (segment (start 122.606 51.4062) (end 131.902 60.7025) (width 0.25) (layer "F.Cu") (net 10))
-  (segment (start 121.884 48.0073) (end 122.606 48.7298) (width 0.25) (layer "F.Cu") (net 10))
-  (segment (start 119.973 49.2) (end 119.973 48.8322) (width 0.25) (layer "F.Cu") (net 10))
-  (segment (start 131.902 60.7025) (end 136.614 60.7025) (width 0.25) (layer "F.Cu") (net 10))
-  (segment (start 122.606 48.7298) (end 122.606 51.4062) (width 0.25) (layer "F.Cu") (net 10))
-  (segment (start 118.796 49.2) (end 119.973 49.2) (width 0.25) (layer "F.Cu") (net 10))
-  (segment (start 120.798 48.0073) (end 121.884 48.0073) (width 0.25) (layer "F.Cu") (net 10))
-  (segment (start 119.973 48.8322) (end 120.798 48.0073) (width 0.25) (layer "F.Cu") (net 10))
-  (segment (start 163.5 87.5882) (end 163.5 97.46) (width 0.25) (layer "F.Cu") (net 10))
-  (segment (start 155.88 51.74) (end 155.88 49.2) (width 0.25) (layer "B.Cu") (net 24))
-  (segment (start 133.02 74.6) (end 155.88 51.74) (width 0.25) (layer "B.Cu") (net 24))
-  (segment (start 144.543 97.8278) (end 144.543 97.46) (width 0.25) (layer "F.Cu") (net 27))
-  (segment (start 126.995 98.6776) (end 143.693 98.6776) (width 0.25) (layer "F.Cu") (net 27))
-  (segment (start 143.693 98.6776) (end 144.543 97.8278) (width 0.25) (layer "F.Cu") (net 27))
-  (segment (start 120.698 92.38) (end 126.995 98.6776) (width 0.25) (layer "F.Cu") (net 27))
-  (segment (start 144.543 97.46) (end 145.72 97.46) (width 0.25) (layer "F.Cu") (net 27))
-  (segment (start 107.62 92.38) (end 120.698 92.38) (width 0.25) (layer "F.Cu") (net 27))
-  (segment (start 130.48 69.52) (end 135.56 74.6) (width 0.25) (layer "F.Cu") (net 29))
-  (segment (start 107.62 69.52) (end 130.48 69.52) (width 0.25) (layer "F.Cu") (net 29))
-  (segment (start 107.62 55.4569) (end 107.62 54.28) (width 0.25) (layer "B.Cu") (net 37))
-  (segment (start 107.254 58.1831) (end 106.426 57.3549) (width 0.25) (layer "B.Cu") (net 37))
-  (segment (start 107.62 58.1831) (end 107.254 58.1831) (width 0.25) (layer "B.Cu") (net 37))
-  (segment (start 107.252 55.4569) (end 107.62 55.4569) (width 0.25) (layer "B.Cu") (net 37))
-  (segment (start 106.426 57.3549) (end 106.426 56.2831) (width 0.25) (layer "B.Cu") (net 37))
-  (segment (start 107.62 59.36) (end 107.62 58.1831) (width 0.25) (layer "B.Cu") (net 37))
-  (segment (start 106.426 56.2831) (end 107.252 55.4569) (width 0.25) (layer "B.Cu") (net 37))
-  (segment (start 107.62 56.82) (end 126.742 56.82) (width 0.25) (layer "F.Cu") (net 39))
-  (segment (start 126.742 56.82) (end 144.522 74.6) (width 0.25) (layer "F.Cu") (net 39))
-  (segment (start 144.522 74.6) (end 145.72 74.6) (width 0.25) (layer "F.Cu") (net 39))
-  (segment (start 127.257 61.9) (end 147.577 82.22) (width 0.25) (layer "F.Cu") (net 40))
-  (segment (start 107.62 61.9) (end 127.257 61.9) (width 0.25) (layer "F.Cu") (net 40))
-  (segment (start 147.577 82.22) (end 155.88 82.22) (width 0.25) (layer "F.Cu") (net 40))
-  (segment (start 132.209 89.84) (end 137.3365 94.9676) (width 0.25) (layer "F.Cu") (net 41))
-  (segment (start 137.3365 94.9676) (end 139.463 97.0942) (width 0.25) (layer "F.Cu") (net 41))
-  (segment (start 139.463 97.0942) (end 139.463 97.46) (width 0.25) (layer "F.Cu") (net 41))
-  (segment (start 137.3365 94.9676) (end 138.5534 94.9676) (width 0.25) (layer "F.Cu") (net 41))
-  (segment (start 107.62 89.84) (end 132.209 89.84) (width 0.25) (layer "F.Cu") (net 41))
-  (segment (start 139.463 97.46) (end 143.18 97.46) (width 0.25) (layer "F.Cu") (net 41))
-  (via (at 138.5534 94.9676) (size 0.6) (drill 0.4) (layers "F.Cu" "B.Cu") (net 41))
-  (segment (start 126.496 50.3769) (end 135.52 59.4002) (width 0.25) (layer "B.Cu") (net 41))
-  (segment (start 135.52 59.4002) (end 135.56 59.36) (width 0.25) (layer "B.Cu") (net 41))
-  (segment (start 131.733 63.1873) (end 135.52 59.4002) (width 0.25) (layer "B.Cu") (net 41))
-  (segment (start 126.416 49.2) (end 126.416 50.3769) (width 0.25) (layer "B.Cu") (net 41))
-  (segment (start 126.416 50.3769) (end 126.496 50.3769) (width 0.25) (layer "B.Cu") (net 41))
-  (segment (start 138.8949 94.538) (end 138.5534 94.8795) (width 0.25) (layer "B.Cu") (net 41))
-  (segment (start 138.895 94.538) (end 138.8949 94.538) (width 0.25) (layer "B.Cu") (net 41))
-  (segment (start 140.64 96.2831) (end 138.895 94.538) (width 0.25) (layer "B.Cu") (net 41))
-  (segment (start 126.496 50.3769) (end 126.577 50.3769) (width 0.25) (layer "B.Cu") (net 41))
-  (segment (start 131.733 87.3758) (end 131.733 63.1873) (width 0.25) (layer "B.Cu") (net 41))
-  (segment (start 138.895 94.538) (end 131.733 87.3758) (width 0.25) (layer "B.Cu") (net 41))
-  (segment (start 140.64 97.46) (end 140.64 96.2831) (width 0.25) (layer "B.Cu") (net 41))
-  (segment (start 138.5534 94.8795) (end 138.5534 94.9676) (width 0.25) (layer "B.Cu") (net 41))
 )
