File: kicad/V1/heaterboard.kicad_sch (KiCad schematic)
At the start: 14 parts, among them J1 Power, J2 Digital/PWM, J3 Analog, J4 Digital/PWM, J5 Screw_Terminal_01x02, J6 Screw_Terminal_01x02, J7 Conn_01x05_Pin, Q1 Q_NMOS_GDS, U1 LM7805_TO220

Commit message: pivot to nano
Parts:
- removed J5: Screw_Terminal_01x02, Connector_PinHeader_2.54mm:PinHeader_1x02_P2.54mm_Vertical, symbol Connector:Screw_Terminal_01x02
- removed TH1: PT100, Connector_JST:JST_XH_B2B-XH-A_1x02_P2.50mm_Vertical, symbol Sensor_Temperature:PT100
- added U2: LM317_TO-220, Package_TO_SOT_THT:TO-220-3_Vertical, symbol Regulator_Linear:LM317_TO-220
Connections:
- net *3: no longer Q1.1 (G)
- net +5V: now also U1.3 (VO)
- net A0: now also R1.2 (-), R2.1 (+)
- net A1: no longer R3.2 (-), R4.1 (+)
- net A3: no longer R1.2 (-), R2.1 (+)
- net GND: now also J7.5 (Pin_5), R4.2 (-), U1.2 (GND)
- net +12V: now reaches J6.2 (Pin_2)
- net +12V: now also J7.2 (Pin_2), J7.4 (Pin_4), R1.1 (+), U1.1 (VI)
- new net: R3.2 (-), R4.1 (+)
- now unconnected: J1.6 (Pin_6), J1.7 (Pin_7)
Other:
- moved on the sheet: J1, J2, J3, J4, J6, J7, Q1, R1, R2, R3, R4, U1
