File: kicad/V2/heaterboard-2.kicad_sch (KiCad schematic)
At the start: 9 parts, among them J1 Screw_Terminal_01x02, J2 Conn_01x05_Pin, Q1 Q_NMOS_GDS, U1 LM317_TO-220

Commit message: to-220
Parts:
- added R5: 0.24 kΩ, Resistor_THT:R_Axial_DIN0207_L6.3mm_D2.5mm_P10.16mm_Horizontal, symbol PCM_Generic:R,IEEE
- added R6: 0.72 kΩ, Resistor_THT:R_Axial_DIN0207_L6.3mm_D2.5mm_P10.16mm_Horizontal, symbol PCM_Generic:R,IEEE
Connections:
- net +12V: now also U1.3 (VI)
- net GND: now also R6.2 (-)
- net at U1.1 (ADJ): now also R5.2 (-), R6.1 (+)
- net +5V: now reaches U1.2 (VO)
- net +5V: now also R5.1 (+)
Other:
- moved on the sheet: U1
Changed lines of the file:
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@@
   (junction (at 111.76 96.52) (diameter 0) (color 0 0 0 0)
   )
+  (junction (at 54.61 38.1) (diameter 0) (color 0 0 0 0)
+  )
   (junction (at 111.76 114.3) (diameter 0) (color 0 0 0 0)
   )
+  (junction (at 54.61 52.07) (diameter 0) (color 0 0 0 0)
+  )
   (junction (at 88.9 101.6) (diameter 0) (color 0 0 0 0)
   )
@@
     (stroke (width 0) (type default))
   )
+  (wire (pts (xy 30.48 38.1) (xy 35.56 38.1))
+    (stroke (width 0) (type default))
+  )
+  (wire (pts (xy 54.61 66.04) (xy 54.61 63.5))
+    (stroke (width 0) (type default))
+  )
+  (wire (pts (xy 43.18 52.07) (xy 54.61 52.07))
+    (stroke (width 0) (type default))
+  )
   (wire (pts (xy 52.07 97.79) (xy 52.07 100.33))
     (stroke (width 0) (type default))
@@
     (stroke (width 0) (type default))
   )
+  (wire (pts (xy 50.8 38.1) (xy 54.61 38.1))
+    (stroke (width 0) (type default))
+  )
+  (wire (pts (xy 54.61 50.8) (xy 54.61 52.07))
+    (stroke (width 0) (type default))
+  )
   (wire (pts (xy 101.6 48.26) (xy 101.6 50.8))
     (stroke (width 0) (type default))
@@
     (stroke (width 0) (type default))
   )
+  (wire (pts (xy 54.61 38.1) (xy 69.85 38.1))
+    (stroke (width 0) (type default))
+  )
   (wire (pts (xy 111.76 104.14) (xy 114.3 104.14))
     (stroke (width 0) (type default))
   )
   (wire (pts (xy 88.9 88.9) (xy 105.41 88.9))
+    (stroke (width 0) (type default))
+  )
+  (wire (pts (xy 54.61 52.07) (xy 54.61 53.34))
+    (stroke (width 0) (type default))
+  )
+  (wire (pts (xy 54.61 38.1) (xy 54.61 40.64))
+    (stroke (width 0) (type default))
+  )
+  (wire (pts (xy 43.18 45.72) (xy 43.18 52.07))
     (stroke (width 0) (type default))
   )
@@
     (effects (font (size 1.27 1.27)) (justify right bottom))
   )
+  (symbol (lib_id "PCM_Generic:R,IEEE") (at 54.61 58.42 0) (unit 1)
+    (in_bom yes) (on_board yes) (dnp no) (fields_autoplaced)
+    (property "Reference" "R6" (at 57.15 55.8799 0)
+      (effects (font (size 2.54 2.54)) (justify left))
+    )
+    (property "Value" "0.72 kΩ" (at 57.15 60.9599 0)
+      (effects (font (size 2.54 2.54)) (justify left))
+    )
+    (property "Footprint" "Resistor_THT:R_Axial_DIN0207_L6.3mm_D2.5mm_P10.16mm_Horizontal" (at 54.61 58.42 0)
+      (effects (font (size 2.54 2.54)) hide)
+    )
+    (property "Datasheet" "" (at 54.61 58.42 0)
+      (effects (font (size 2.54 2.54)) hide)
+    )
+    (property "Indicator" "+" (at 52.07 55.88 0)
+      (effects (font (size 1.27 1.27)) hide)
+    )
+    (pin "1")
+    (pin "2")
+    (instances
+      (project "heaterboard-2"
+        (path "/63b0bf45-0e24-4f26-a68d-dac5d63dd697"
+          (reference "R6") (unit 1)
+        )
+      )
+    )
+  )
+  (symbol (lib_id "PCM_Generic:R,IEEE") (at 54.61 45.72 0) (unit 1)
+    (in_bom yes) (on_board yes) (dnp no) (fields_autoplaced)
+    (property "Reference" "R5" (at 57.15 43.1799 0)
+      (effects (font (size 2.54 2.54)) (justify left))
+    )
+    (property "Value" "0.24 kΩ" (at 57.15 48.2599 0)
+      (effects (font (size 2.54 2.54)) (justify left))
+    )
+    (property "Footprint" "Resistor_THT:R_Axial_DIN0207_L6.3mm_D2.5mm_P10.16mm_Horizontal" (at 54.61 45.72 0)
+      (effects (font (size 2.54 2.54)) hide)
+    )
+    (property "Datasheet" "" (at 54.61 45.72 0)
+      (effects (font (size 2.54 2.54)) hide)
+    )
+    (property "Indicator" "+" (at 52.07 43.18 0)
+      (effects (font (size 1.27 1.27)) hide)
+    )
+    (pin "1")
+    (pin "2")
+    (instances
+      (project "heaterboard-2"
+        (path "/63b0bf45-0e24-4f26-a68d-dac5d63dd697"
+          (reference "R5") (unit 1)
+        )
+      )
+    )
+  )
+  (symbol (lib_id "power:+12V") (at 30.48 38.1 0) (unit 1)
+    (in_bom yes) (on_board yes) (dnp no) (fields_autoplaced)
+    (property "Reference" "#PWR08" (at 30.48 41.91 0)
+      (effects (font (size 1.27 1.27)) hide)
+    )
+    (property "Value" "+12V" (at 30.48 33.02 0)
+      (effects (font (size 1.27 1.27)))
+    )
+    (property "Footprint" "" (at 30.48 38.1 0)
+      (effects (font (size 1.27 1.27)) hide)
+    )
+    (property "Datasheet" "" (at 30.48 38.1 0)
+      (effects (font (size 1.27 1.27)) hide)
+    )
+    (pin "1")
+    (instances
+      (project "heaterboard-2"
+        (path "/63b0bf45-0e24-4f26-a68d-dac5d63dd697"
+          (reference "#PWR08") (unit 1)
+        )
+      )
+    )
+  )
   (symbol (lib_id "PCM_Generic:R,IEEE") (at 101.6 40.64 0) (unit 1)
     (in_bom yes) (on_board yes) (dnp no) (fields_autoplaced)
@@
     )
   )
-  (symbol (lib_id "Regulator_Linear:LM317_TO-220") (at 50.8 38.1 0) (unit 1)
-    (in_bom yes) (on_board yes) (dnp no) (fields_autoplaced)
-    (property "Reference" "U1" (at 50.8 31.75 0)
-      (effects (font (size 1.27 1.27)))
-    )
-    (property "Value" "LM317_TO-220" (at 50.8 34.29 0)
-      (effects (font (size 1.27 1.27)))
-    )
-    (property "Footprint" "Package_TO_SOT_THT:TO-220-3_Vertical" (at 50.8 31.75 0)
+  (symbol (lib_id "power:+5V") (at 69.85 38.1 0) (unit 1)
+    (in_bom yes) (on_board yes) (dnp no) (fields_autoplaced)
+    (property "Reference" "#PWR09" (at 69.85 41.91 0)
+      (effects (font (size 1.27 1.27)) hide)
+    )
+    (property "Value" "+5V" (at 69.85 33.02 0)
+      (effects (font (size 1.27 1.27)))
+    )
+    (property "Footprint" "" (at 69.85 38.1 0)
+      (effects (font (size 1.27 1.27)) hide)
+    )
+    (property "Datasheet" "" (at 69.85 38.1 0)
+      (effects (font (size 1.27 1.27)) hide)
+    )
+    (pin "1")
+    (instances
+      (project "heaterboard-2"
+        (path "/63b0bf45-0e24-4f26-a68d-dac5d63dd697"
+          (reference "#PWR09") (unit 1)
+        )
+      )
+    )
+  )
+  (symbol (lib_id "Regulator_Linear:LM317_TO-220") (at 43.18 38.1 0) (unit 1)
+    (in_bom yes) (on_board yes) (dnp no) (fields_autoplaced)
+    (property "Reference" "U1" (at 43.18 31.75 0)
+      (effects (font (size 1.27 1.27)))
+    )
+    (property "Value" "LM317_TO-220" (at 43.18 34.29 0)
+      (effects (font (size 1.27 1.27)))
+    )
+    (property "Footprint" "Package_TO_SOT_THT:TO-220-3_Vertical" (at 43.18 31.75 0)
       (effects (font (size 1.27 1.27) italic) hide)
     )
-    (property "Datasheet" "http://www.ti.com/lit/ds/symlink/lm317.pdf" (at 50.8 38.1 0)
+    (property "Datasheet" "http://www.ti.com/lit/ds/symlink/lm317.pdf" (at 43.18 38.1 0)
       (effects (font (size 1.27 1.27)) hide)
     )
@@
         )
       )
+    )
+  )
+  (symbol (lib_name "GND_1") (lib_id "power:GND") (at 54.61 66.04 0) (unit 1)
+    (in_bom yes) (on_board yes) (dnp no) (fields_autoplaced)
+    (property "Reference" "#PWR010" (at 54.61 72.39 0)
+      (effects (font (size 1.27 1.27)) hide)
+    )
+    (property "Value" "GND" (at 54.61 71.12 0)
+      (effects (font (size 1.27 1.27)))
+    )
+    (property "Footprint" "" (at 54.61 66.04 0)
+      (effects (font (size 1.27 1.27)) hide)
+    )
+    (property "Datasheet" "" (at 54.61 66.04 0)
+      (effects (font (size 1.27 1.27)) hide)
+    )
+    (pin "1")
+    (instances
+      (project "heaterboard-2"
+        (path "/63b0bf45-0e24-4f26-a68d-dac5d63dd697"
+          (reference "#PWR010") (unit 1)
+        )
+      )

Commit message: 220
Other:
- note added: "66666"
Changed lines of the file:
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@@
+    (effects (font (size 1.27 1.27)) (justify left bottom))
+  )
+  (text "66666" (at 33.02 68.58 0)
     (effects (font (size 1.27 1.27)) (justify left bottom))
   )
