File: kicad/V2/heaterboard-2.kicad_sch (KiCad schematic)
At the start: 10 parts, among them J1 Screw_Terminal_01x02, J2 Conn_01x05_Pin, Q1 Q_NMOS_GDS, U1 LM317_TO-220, U2 LM7805_TO220

Commit message: End of class 1 feb
Parts:
- removed U2: LM7805_TO220, Package_TO_SOT_THT:TO-220-3_Vertical, symbol Regulator_Linear:LM7805_TO220
Connections:
- net A0: now also A1.A0
- net GND: now also A1.GND2 (GND), Q1.3 (S)
- net A1: now reaches A1.A1
- net A1: now also R3.2 (-), R4.1 (+)
- net A2: now reaches A1.A2
- net A3: now reaches A1.A3
- net A4: now reaches A1.A4 (A4/SDA)
- net A5: now reaches A1.A5 (A5/SCL)
- net A6: now reaches A1.A6
- net A7: now reaches A1.A7
- net AREF: now reaches A1.AREF
- net D0: now reaches A1.D0 (D0/RX)
- net D1: now reaches A1.D1 (D1/TX)
- net D10: now reaches A1.D10
- net D11: now reaches A1.D11 (D11_MOSI)
- net D12: now reaches A1.D12 (D12_MISO)
- net D13: now reaches A1.D13 (D13_SCK)
- net D2: now reaches A1.D2 (D2_INT0)
- net D3: now reaches A1.D3 (D3_INT1)
- net D4: now reaches A1.D4
- net D5: now reaches A1.D5
- net D6: now reaches A1.D6
- net D7: now reaches A1.D7
- net D8: now reaches A1.D8
- net D9: now reaches A1.D9
Other:
- note added: "BATTERY VOLTAGE MONITOR"
- note added: "BOARD POWER REGULATION"
- note added: "HEATER POWER CONTROL"
- note added: "WIRELESS RELAY"
- note added: "Wikipedia - LM317"
- company: (none) -> ME692
- title: (none) -> Windshield Heater
- moved on the sheet: A1, J1, J2, Q1, R1, R2, R3, R4, U1

Commit message: 111
Parts:
- added J3: Conn_01x04_Pin, symbol Connector:Conn_01x04_Pin
- added R5: 0.4 kΩ, Resistor_THT:R_Axial_DIN0207_L6.3mm_D2.5mm_P10.16mm_Horizontal, symbol PCM_Generic:R,IEEE
- added R6: 2.4 kΩ, Resistor_THT:R_Axial_DIN0207_L6.3mm_D2.5mm_P10.16mm_Horizontal, symbol PCM_Generic:R,IEEE
Connections:
- net +12V: now also U1.3 (VI)
- net A4: now also J3.4 (Pin_4)
- net A5: now also J3.3 (Pin_3)
- net D9: now also Q1.1 (G)
- net GND: now also J3.2 (Pin_2), R6.2 (-)
- net at U1.1 (ADJ): now also R5.2 (-), R6.1 (+)
- net +9V: now reaches U1.2 (VO)
- net +9V: now also A1.VIN, R5.1 (+)
- new net +5V: J3.1 (Pin_1)
Other:
- note added: "66666"
- note added: "LM317 Calculator"
- note added: "TEMPERATURE MODULE"
- moved on the sheet: U1

Commit message: pcb stuff
Parts:
- J3: footprint (none) -> Connector_PinSocket_2.54mm:PinSocket_1x04_P2.54mm_Vertical
Other:
- note added: "Amazon"
Changed lines of the file:
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@@
     (effects (font (size 1.27 1.27)) (justify left bottom))
+  )
+  (text "Amazon" (at 26.67 129.54 0)
+    (effects (font (size 1.27 1.27)) (justify left bottom) (href "https://www.amazon.com/HiLetgo-Precision-Temperature-Humidity-2-0-5-5V/dp/B09KGW1G41"))
   )
   (text "66666" (at 33.02 68.58 0)
@@
       (effects (font (size 1.27 1.27)))
     )
-    (property "Footprint" "" (at 41.91 147.32 0)
-      (effects (font (size 1.27 1.27)) hide)
-    )
+    (property "Footprint" "Connector_PinSocket_2.54mm:PinSocket_1x04_P2.54mm_Vertical" (at 41.91 147.32 0)
+      (effects (font (size 1.27 1.27)) hide)
+    )

Commit message: end class02-06-2024
Parts:
- added C1: 100nF, symbol Device:C
- added C2: 1μF, symbol Device:C_Polarized_US
- R5: value 0.4 kΩ -> 0.4kΩ
- R6: value 2.4 kΩ -> 2.4kΩ
Connections:
- net +12V: now also C1.1
- net +9V: now also C2.1
- net GND: now also C1.2, C2.2
Other:
- note removed: "66666"
- moved on the sheet: R5, R6, U1

Commit message: pcb layout
Parts:
- C1, C2: footprint (none) -> Capacitor_THT:CP_Radial_D10.0mm_P5.00mm
- J1: footprint Connector_PinHeader_2.54mm:PinHeader_1x02_P2.54mm_Vertical -> TerminalBlock:TerminalBlock_Wuerth_691311400102_P7.62mm
Other:
- title: Windshield Heater -> Windshield Heater Controller Schematic
Changed lines of the file:
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@@
   (paper "USLetter")
   (title_block
-    (title "Windshield Heater")
+    (title "Windshield Heater Controller Schematic")
     (rev "2")
     (company "ME692")
@@
       (effects (font (size 1.27 1.27)) (justify left))
     )
-    (property "Footprint" "" (at 67.31 55.88 0)
+    (property "Footprint" "Capacitor_THT:CP_Radial_D10.0mm_P5.00mm" (at 67.31 55.88 0)
       (effects (font (size 1.27 1.27)) hide)
     )
@@
       (effects (font (size 1.27 1.27)) (justify left))
     )
-    (property "Footprint" "" (at 33.9852 59.69 0)
+    (property "Footprint" "Capacitor_THT:CP_Radial_D10.0mm_P5.00mm" (at 33.9852 59.69 0)
       (effects (font (size 1.27 1.27)) hide)
     )
@@
       (effects (font (size 1.27 1.27)))
     )
-    (property "Footprint" "Connector_PinHeader_2.54mm:PinHeader_1x02_P2.54mm_Vertical" (at 46.99 97.79 0)
-      (effects (font (size 1.27 1.27)) hide)
-    )
+    (property "Footprint" "TerminalBlock:TerminalBlock_Wuerth_691311400102_P7.62mm" (at 46.99 97.79 0)
+      (effects (font (size 1.27 1.27)) hide)
+    )

Commit message: pcb layout and began routing
Parts:
- added J1: Screw_Terminal_01x02, Connector_Molex:Molex_Mega-Fit_76825-0002_2x01_P5.70mm_Horizontal, symbol Connector:Screw_Terminal_01x02
- J2: renamed from J1; footprint TerminalBlock:TerminalBlock_Wuerth_691311400102_P7.62mm -> Connector_Molex:Molex_Mega-Fit_76825-0002_2x01_P5.70mm_Horizontal
- J3: footprint Connector_PinSocket_2.54mm:PinSocket_1x04_P2.54mm_Vertical -> Connector_Molex:Molex_Micro-Fit_3.0_43650-0400_1x04_P3.00mm_Horizontal
- J4: renamed from J2; footprint Connector_PinHeader_2.54mm:PinHeader_1x05_P2.54mm_Vertical -> Connector_Molex:Molex_Micro-Fit_3.0_43650-0515_1x05_P3.00mm_Vertical
- R1: renamed from R5; symbol PCM_Generic:R,IEEE -> Device:R_US
- R2: renamed from R6; symbol PCM_Generic:R,IEEE -> Device:R_US
- R3: renamed from R1; symbol PCM_Generic:R,IEEE -> Device:R_US
- R4: renamed from R2; symbol PCM_Generic:R,IEEE -> Device:R_US
- R5: renamed from R3; symbol PCM_Generic:R,IEEE -> Device:R_US
- R6: renamed from R4; symbol PCM_Generic:R,IEEE -> Device:R_US
Connections:
- net +12V: now also J1.2 (Pin_2)
- net GND: now also R4.2, J1.1 (Pin_1)
Other:
- note added: "Amazon - RF control module"
- note added: "Amazon - Temp module"
- note added: "POWER INPUT"
- note removed: "Amazon"
- note removed: "RF control module link"
- moved on the sheet: C1, C2, J2, J4, U1

Commit message: end of class 15 feb
Parts:
- C1: footprint Capacitor_THT:CP_Radial_D10.0mm_P5.00mm -> Capacitor_SMD:C_1206_3216Metric_Pad1.33x1.80mm_HandSolder; Catalog No (none) -> 478-KAM31BR71H104KTCT-ND; Vendor (none) -> Digikey
- C2: footprint Capacitor_THT:CP_Radial_D10.0mm_P5.00mm -> Capacitor_SMD:C_1206_3216Metric_Pad1.33x1.80mm_HandSolder
- R1, R2, R3, R4, R5, R6: footprint Resistor_THT:R_Axial_DIN0207_L6.3mm_D2.5mm_P10.16mm_Horizontal -> Resistor_SMD:R_1206_3216Metric_Pad1.30x1.75mm_HandSolder
Changed lines of the file:
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@@
       (effects (font (size 2.54 2.54)) (justify left))
     )
-    (property "Footprint" "Resistor_THT:R_Axial_DIN0207_L6.3mm_D2.5mm_P10.16mm_Horizontal" (at 102.616 57.404 90)
+    (property "Footprint" "Resistor_SMD:R_1206_3216Metric_Pad1.30x1.75mm_HandSolder" (at 102.616 57.404 90)
       (effects (font (size 1.27 1.27)) hide)
     )
@@
       (effects (font (size 2.54 2.54)) (justify left))
     )
-    (property "Footprint" "Resistor_THT:R_Axial_DIN0207_L6.3mm_D2.5mm_P10.16mm_Horizontal" (at 102.616 44.704 90)
+    (property "Footprint" "Resistor_SMD:R_1206_3216Metric_Pad1.30x1.75mm_HandSolder" (at 102.616 44.704 90)
       (effects (font (size 1.27 1.27)) hide)
     )
@@
       (effects (font (size 2.54 2.54)) (justify left))
     )
-    (property "Footprint" "Resistor_THT:R_Axial_DIN0207_L6.3mm_D2.5mm_P10.16mm_Horizontal" (at 98.806 92.964 90)
+    (property "Footprint" "Resistor_SMD:R_1206_3216Metric_Pad1.30x1.75mm_HandSolder" (at 98.806 92.964 90)
       (effects (font (size 1.27 1.27)) hide)
     )
@@
       (effects (font (size 1.27 1.27)) (justify left))
     )
-    (property "Footprint" "Capacitor_THT:CP_Radial_D10.0mm_P5.00mm" (at 118.11 55.88 0)
+    (property "Footprint" "Capacitor_SMD:C_1206_3216Metric_Pad1.33x1.80mm_HandSolder" (at 118.11 55.88 0)
       (effects (font (size 1.27 1.27)) hide)
     )
@@
       (effects (font (size 2.54 2.54)) (justify left))
     )
-    (property "Footprint" "Resistor_THT:R_Axial_DIN0207_L6.3mm_D2.5mm_P10.16mm_Horizontal" (at 98.806 108.204 90)
+    (property "Footprint" "Resistor_SMD:R_1206_3216Metric_Pad1.30x1.75mm_HandSolder" (at 98.806 108.204 90)
       (effects (font (size 1.27 1.27)) hide)
     )
@@
       (effects (font (size 1.27 1.27)) (justify left))
     )
-    (property "Footprint" "Capacitor_THT:CP_Radial_D10.0mm_P5.00mm" (at 84.7852 59.69 0)
+    (property "Footprint" "Capacitor_SMD:C_1206_3216Metric_Pad1.33x1.80mm_HandSolder" (at 84.7852 59.69 0)
       (effects (font (size 1.27 1.27)) hide)
     )
     (property "Datasheet" "~" (at 83.82 55.88 0)
+      (effects (font (size 1.27 1.27)) hide)
+    )
+    (property "Catalog No" "478-KAM31BR71H104KTCT-ND" (at 83.82 55.88 0)
+      (effects (font (size 1.27 1.27)) hide)
+    )
+    (property "Vendor" "Digikey" (at 83.82 55.88 0)
       (effects (font (size 1.27 1.27)) hide)
     )
@@
       (effects (font (size 2.54 2.54)) (justify left))
     )
-    (property "Footprint" "Resistor_THT:R_Axial_DIN0207_L6.3mm_D2.5mm_P10.16mm_Horizontal" (at 89.916 159.004 90)
+    (property "Footprint" "Resistor_SMD:R_1206_3216Metric_Pad1.30x1.75mm_HandSolder" (at 89.916 159.004 90)
       (effects (font (size 1.27 1.27)) hide)
     )
@@
       (effects (font (size 2.54 2.54)) (justify left))
     )
-    (property "Footprint" "Resistor_THT:R_Axial_DIN0207_L6.3mm_D2.5mm_P10.16mm_Horizontal" (at 89.916 146.304 90)
-      (effects (font (size 1.27 1.27)) hide)
-    )
+    (property "Footprint" "Resistor_SMD:R_1206_3216Metric_Pad1.30x1.75mm_HandSolder" (at 89.916 146.304 90)
+      (effects (font (size 1.27 1.27)) hide)
+    )

Commit message: more update
Parts:
- C2: symbol Device:C_Polarized_US -> Device:C
Changed lines of the file:
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@@
     )
   )
-  (symbol (lib_id "Device:C_Polarized_US") (at 118.11 55.88 0) (unit 1)
+  (symbol (lib_id "Device:C") (at 118.11 55.88 0) (unit 1)
     (in_bom yes) (on_board yes) (dnp no)
     (property "Reference" "C2" (at 121.92 53.975 0)
@@
       (effects (font (size 1.27 1.27)) (justify left))
     )
-    (property "Footprint" "Capacitor_SMD:C_1206_3216Metric_Pad1.33x1.80mm_HandSolder" (at 118.11 55.88 0)
+    (property "Footprint" "Capacitor_SMD:C_1206_3216Metric_Pad1.33x1.80mm_HandSolder" (at 119.0752 59.69 0)
       (effects (font (size 1.27 1.27)) hide)
     )
