File: kicad/V2/heaterboard-2.kicad_sch (KiCad schematic)
At the start: 15 parts, among them J1 Screw_Terminal_01x02, J2 Screw_Terminal_01x02, J3 Conn_01x04_Pin, J4 Conn_01x05_Pin, Q1 Q_NMOS_GDS, U1 LM317_TO-220

Commit message: Catalog No Update
Catalog No Update
Parts:
- C2: Catalog No (none) -> 490-KRM31KR72A105KH01KCT-ND; Vendor (none) -> Digikey
- J1, J2: Catalog No (none) -> WM11969-ND; Vendor (none) -> Digikey
- J3: Catalog No (none) -> WM1862-ND; Vendor (none) -> Digikey
- J4: Catalog No (none) -> WM1920-ND; Vendor (none) -> Digikey
- R1: Catalog No (none) -> 13-RT1206BRD07400RLCT-ND; Vendor (none) -> Digikey
- R2: Catalog No (none) -> 13-RC0603FR-132K4LCT-ND; Vendor (none) -> Digikey
- R3: Catalog No (none) -> 311-10.0KLRCT-ND; Vendor (none) -> Digikey
- R4, R6: Catalog No (none) -> 13-RT0603BRE075KLCT-ND; Vendor (none) -> Digikey
- R5: Catalog No (none) -> YAG2302CT-ND; Vendor (none) -> Digikey
Changed lines of the file:
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@@
+      (effects (font (size 1.27 1.27)) hide)
+    )
+    (property "Catalog No" "13-RC0603FR-132K4LCT-ND" (at 101.6 57.15 0)
+      (effects (font (size 1.27 1.27)) hide)
+    )
+    (property "Vendor" "Digikey" (at 101.6 57.15 0)
       (effects (font (size 1.27 1.27)) hide)
     )
@@
       (effects (font (size 1.27 1.27)) hide)
     )
+    (property "Catalog No" "13-RT1206BRD07400RLCT-ND" (at 101.6 44.45 0)
+      (effects (font (size 1.27 1.27)) hide)
+    )
+    (property "Vendor" "Digikey" (at 101.6 44.45 0)
+      (effects (font (size 1.27 1.27)) hide)
+    )
     (pin "1")
     (pin "2")
@@
     )
     (property "Indicator" "+" (at 95.25 90.17 0)
+      (effects (font (size 1.27 1.27)) hide)
+    )
+    (property "Catalog No" "311-10.0KLRCT-ND" (at 97.79 92.71 0)
+      (effects (font (size 1.27 1.27)) hide)
+    )
+    (property "Vendor" "Digikey" (at 97.79 92.71 0)
       (effects (font (size 1.27 1.27)) hide)
     )
@@
       (effects (font (size 1.27 1.27)) hide)
     )
+    (property "Catalog No" "490-KRM31KR72A105KH01KCT-ND" (at 118.11 55.88 0)
+      (effects (font (size 1.27 1.27)) hide)
+    )
+    (property "Vendor" "Digikey" (at 118.11 55.88 0)
+      (effects (font (size 1.27 1.27)) hide)
+    )
     (pin "1")
     (pin "2")
@@
       (effects (font (size 1.27 1.27)) hide)
     )
+    (property "Catalog No" "WM1920-ND" (at 119.38 149.86 0)
+      (effects (font (size 1.27 1.27)) hide)
+    )
+    (property "Vendor" "Digikey" (at 119.38 149.86 0)
+      (effects (font (size 1.27 1.27)) hide)
+    )
     (pin "4")
     (pin "2")
@@
       (effects (font (size 1.27 1.27)) hide)
     )
+    (property "Catalog No" "13-RT0603BRE075KLCT-ND" (at 97.79 107.95 0)
+      (effects (font (size 1.27 1.27)) hide)
+    )
+    (property "Vendor" "Digikey" (at 97.79 107.95 0)
+      (effects (font (size 1.27 1.27)) hide)
+    )
     (pin "1")
     (pin "2")
@@
     )
     (property "Datasheet" "https://www.molex.com/en-us/products/part-detail/768250002?display=pdf" (at 40.64 41.91 0)
+      (effects (font (size 1.27 1.27)) hide)
+    )
+    (property "Catalog No" "WM11969-ND" (at 40.64 41.91 0)
+      (effects (font (size 1.27 1.27)) hide)
+    )
+    (property "Vendor" "Digikey" (at 40.64 41.91 0)
       (effects (font (size 1.27 1.27)) hide)
     )
@@
     )
     (property "Datasheet" "https://www.molex.com/en-us/products/part-detail/768250002?display=pdf" (at 39.37 97.79 0)
+      (effects (font (size 1.27 1.27)) hide)
+    )
+    (property "Catalog No" "WM11969-ND" (at 39.37 97.79 0)
+      (effects (font (size 1.27 1.27)) hide)
+    )
+    (property "Vendor" "Digikey" (at 39.37 97.79 0)
       (effects (font (size 1.27 1.27)) hide)
     )
@@
       (effects (font (size 1.27 1.27)) hide)
     )
+    (property "Catalog No" "13-RT0603BRE075KLCT-ND" (at 88.9 158.75 0)
+      (effects (font (size 1.27 1.27)) hide)
+    )
+    (property "Vendor" "Digikey" (at 88.9 158.75 0)
+      (effects (font (size 1.27 1.27)) hide)
+    )
     (pin "1")
     (pin "2")
@@
     )
     (property "Datasheet" "~" (at 41.91 147.32 0)
+      (effects (font (size 1.27 1.27)) hide)
+    )
+    (property "Catalog No" "WM1862-ND" (at 41.91 147.32 0)
+      (effects (font (size 1.27 1.27)) hide)
+    )
+    (property "Vendor" "Digikey" (at 41.91 147.32 0)
       (effects (font (size 1.27 1.27)) hide)
     )
@@
       (effects (font (size 1.27 1.27)) hide)
     )
+    (property "Catalog No" "YAG2302CT-ND" (at 88.9 146.05 0)
+      (effects (font (size 1.27 1.27)) hide)
+    )
+    (property "Vendor" "Digikey" (at 88.9 146.05 0)
+      (effects (font (size 1.27 1.27)) hide)
+    )

Commit message: Routing, parts, bom
Parts:
- C1: Catalog No 478-KAM31BR71H104KTCT-ND -> 445-12839-1-ND
- C2: Catalog No 490-KRM31KR72A105KH01KCT-ND -> 445-5702-1-ND
- J1: value Screw_Terminal_01x02 -> Power In
- J2: value Screw_Terminal_01x02 -> Heater Connect
- J3: value Conn_01x04_Pin -> Temp Sensor
- J4: value Conn_01x05_Pin -> Relay
- Q1: Catalog No 74AH1189 -> 1727-5291-ND; Vendor Newark -> Digikey
- R1: Catalog No 13-RT1206BRD07400RLCT-ND -> 13-RT1206BRD07400RLDKR-ND
- R2: Catalog No 13-RC0603FR-132K4LCT-ND -> 13-RT1206BRD072K4LCT-ND
- R3: Catalog No 311-10.0KLRCT-ND -> YAG1242CT-ND
- R4, R6: Catalog No 13-RT0603BRE075KLCT-ND -> YAG5090CT-ND
- R5: Catalog No YAG2302CT-ND -> 13-RT1206FRE0715KLCT-ND
- U1: Catalog No (none) -> 296-13869-5-ND; Vendor (none) -> Digikey
Connections:
- net A0: no longer R3.2, R4.1
- net A1: no longer R5.2, R6.1
- net A6: now also R3.2, R4.1
- net A7: now also R5.2, R6.1
Changed lines of the file:
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@@
     (effects (font (size 1.27 1.27)) (justify left bottom))
   )
-  (label "A1" (at 83.82 152.4 180) (fields_autoplaced)
+  (label "A7" (at 83.82 152.4 180) (fields_autoplaced)
     (effects (font (size 1.27 1.27)) (justify right bottom))
   )
@@
     (effects (font (size 1.27 1.27)) (justify left bottom))
   )
-  (label "A0" (at 110.49 100.33 0) (fields_autoplaced)
+  (label "A6" (at 110.49 100.33 0) (fields_autoplaced)
     (effects (font (size 1.27 1.27)) (justify left bottom))
   )
@@
       (effects (font (size 1.27 1.27)) hide)
     )
-    (property "Datasheet" "~" (at 101.6 57.15 0)
+    (property "Datasheet" "https://www.yageo.com/upload/media/product/app/datasheet/rchip/pyu-rt_1-to-0.01_rohs_l.pdf" (at 101.6 57.15 0)
       (effects (font (size 1.27 1.27)) hide)
     )
@@
       (effects (font (size 1.27 1.27)) hide)
     )
-    (property "Catalog No" "13-RC0603FR-132K4LCT-ND" (at 101.6 57.15 0)
+    (property "Catalog No" "13-RT1206BRD072K4LCT-ND" (at 101.6 57.15 0)
       (effects (font (size 1.27 1.27)) hide)
     )
@@
       (effects (font (size 1.27 1.27)) hide)
     )
-    (property "Datasheet" "~" (at 101.6 44.45 0)
+    (property "Datasheet" "https://www.yageo.com/upload/media/product/app/datasheet/rchip/pyu-rt_1-to-0.01_rohs_l.pdf" (at 101.6 44.45 0)
       (effects (font (size 1.27 1.27)) hide)
     )
@@
       (effects (font (size 1.27 1.27)) hide)
     )
-    (property "Catalog No" "13-RT1206BRD07400RLCT-ND" (at 101.6 44.45 0)
+    (property "Catalog No" "13-RT1206BRD07400RLDKR-ND" (at 101.6 44.45 0)
       (effects (font (size 1.27 1.27)) hide)
     )
@@
       (effects (font (size 1.27 1.27)) hide)
     )
-    (property "Datasheet" "~" (at 97.79 92.71 0)
+    (property "Datasheet" "https://www.yageo.com/upload/media/product/app/datasheet/rchip/pyu-rt_1-to-0.01_rohs_l.pdf" (at 97.79 92.71 0)
       (effects (font (size 1.27 1.27)) hide)
     )
@@
       (effects (font (size 1.27 1.27)) hide)
     )
-    (property "Catalog No" "311-10.0KLRCT-ND" (at 97.79 92.71 0)
+    (property "Catalog No" "YAG1242CT-ND" (at 97.79 92.71 0)
       (effects (font (size 1.27 1.27)) hide)
     )
@@
     )
     (property "Datasheet" "http://www.ti.com/lit/ds/symlink/lm317.pdf" (at 92.71 38.1 0)
+      (effects (font (size 1.27 1.27)) hide)
+    )
+    (property "Catalog No" "296-13869-5-ND" (at 92.71 38.1 0)
+      (effects (font (size 1.27 1.27)) hide)
+    )
+    (property "Vendor" "Digikey" (at 92.71 38.1 0)
       (effects (font (size 1.27 1.27)) hide)
     )
@@
       (effects (font (size 1.27 1.27)) hide)
     )
-    (property "Datasheet" "~" (at 118.11 55.88 0)
-      (effects (font (size 1.27 1.27)) hide)
-    )
-    (property "Catalog No" "490-KRM31KR72A105KH01KCT-ND" (at 118.11 55.88 0)
+    (property "Datasheet" "https://product.tdk.com/system/files/dam/doc/product/capacitor/ceramic/mlcc/catalog/mlcc_automotive_general_en.pdf" (at 118.11 55.88 0)
+      (effects (font (size 1.27 1.27)) hide)
+    )
+    (property "Catalog No" "445-5702-1-ND" (at 118.11 55.88 0)
       (effects (font (size 1.27 1.27)) hide)
     )
@@
       (effects (font (size 1.27 1.27)))
     )
-    (property "Value" "Conn_01x05_Pin" (at 118.745 142.24 0)
+    (property "Value" "Relay" (at 118.745 142.24 0)
       (effects (font (size 1.27 1.27)))
     )
@@
       (effects (font (size 1.27 1.27)) hide)
     )
-    (property "Datasheet" "~" (at 119.38 149.86 0)
+    (property "Datasheet" "https://tools.molex.com/pdm_docs/sd/436500515_sd.pdf" (at 119.38 149.86 0)
       (effects (font (size 1.27 1.27)) hide)
     )
@@
       (effects (font (size 1.27 1.27)) hide)
     )
-    (property "Datasheet" "~" (at 97.79 107.95 0)
+    (property "Datasheet" "https://www.yageo.com/upload/media/product/app/datasheet/rchip/pyu-rt_1-to-0.01_rohs_l.pdf" (at 97.79 107.95 0)
       (effects (font (size 1.27 1.27)) hide)
     )
@@
       (effects (font (size 1.27 1.27)) hide)
     )
-    (property "Catalog No" "13-RT0603BRE075KLCT-ND" (at 97.79 107.95 0)
+    (property "Catalog No" "YAG5090CT-ND" (at 97.79 107.95 0)
       (effects (font (size 1.27 1.27)) hide)
     )
@@
       (effects (font (size 1.27 1.27)) (justify right))
     )
-    (property "Value" "Screw_Terminal_01x02" (at 45.72 43.18 90)
+    (property "Value" "Power In" (at 45.72 43.18 90)
       (effects (font (size 1.27 1.27)) (justify right))
     )
@@
       (effects (font (size 1.27 1.27)) hide)
     )
-    (property "Datasheet" "https://www.molex.com/en-us/products/part-detail/768250002?display=pdf" (at 40.64 41.91 0)
+    (property "Datasheet" "https://mm.digikey.com/Volume0/opasdata/d220001/medias/docus/1100/Mega-Fit_Power_Conn.pdf" (at 40.64 41.91 0)
       (effects (font (size 1.27 1.27)) hide)
     )
@@
       (effects (font (size 1.27 1.27)) hide)
     )
-    (property "Datasheet" "~" (at 83.82 55.88 0)
-      (effects (font (size 1.27 1.27)) hide)
-    )
-    (property "Catalog No" "478-KAM31BR71H104KTCT-ND" (at 83.82 55.88 0)
+    (property "Datasheet" "https://product.tdk.com/system/files/dam/doc/product/capacitor/ceramic/mlcc/catalog/mlcc_automotive_general_en.pdf" (at 83.82 55.88 0)
+      (effects (font (size 1.27 1.27)) hide)
+    )
+    (property "Catalog No" "445-12839-1-ND" (at 83.82 55.88 0)
       (effects (font (size 1.27 1.27)) hide)
     )
@@
       (effects (font (size 1.27 1.27)))
     )
-    (property "Value" "Screw_Terminal_01x02" (at 39.37 91.44 0)
+    (property "Value" "Heater Connect" (at 39.37 91.44 0)
       (effects (font (size 1.27 1.27)))
     )
@@
       (effects (font (size 1.27 1.27)) hide)
     )
-    (property "Datasheet" "https://www.molex.com/en-us/products/part-detail/768250002?display=pdf" (at 39.37 97.79 0)
+    (property "Datasheet" "https://mm.digikey.com/Volume0/opasdata/d220001/medias/docus/1100/Mega-Fit_Power_Conn.pdf" (at 39.37 97.79 0)
       (effects (font (size 1.27 1.27)) hide)
     )
@@
       (effects (font (size 1.27 1.27)) hide)
     )
-    (property "Datasheet" "https://4donline.ihs.com/images/VipMasterIC/IC/NEXP/NEXP-S-A0003060256/NEXP-S-A0003059732-1.pdf?hkey=6D3A4C79FDBF58556ACFDE234799DDF0" (at 49.53 105.41 0)
-      (effects (font (size 1.27 1.27)) hide)
-    )
-    (property "Catalog No" "74AH1189 " (at 49.53 105.41 0)
-      (effects (font (size 1.27 1.27)) hide)
-    )
-    (property "Vendor" "Newark" (at 49.53 105.41 0)
+    (property "Datasheet" "https://assets.nexperia.com/documents/data-sheet/PSMN1R1-30PL.pdf" (at 49.53 105.41 0)
+      (effects (font (size 1.27 1.27)) hide)
+    )
+    (property "Catalog No" "1727-5291-ND" (at 49.53 105.41 0)
+      (effects (font (size 1.27 1.27)) hide)
+    )
+    (property "Vendor" "Digikey" (at 49.53 105.41 0)
       (effects (font (size 1.27 1.27)) hide)
     )
@@
       (effects (font (size 1.27 1.27)) hide)
     )
-    (property "Datasheet" "~" (at 88.9 158.75 0)
+    (property "Datasheet" "https://www.yageo.com/upload/media/product/app/datasheet/rchip/pyu-rt_1-to-0.01_rohs_l.pdf" (at 88.9 158.75 0)
       (effects (font (size 1.27 1.27)) hide)
     )
@@
       (effects (font (size 1.27 1.27)) hide)
     )
-    (property "Catalog No" "13-RT0603BRE075KLCT-ND" (at 88.9 158.75 0)
+    (property "Catalog No" "YAG5090CT-ND" (at 88.9 158.75 0)
       (effects (font (size 1.27 1.27)) hide)
     )
@@
       (effects (font (size 1.27 1.27)))
     )
-    (property "Value" "Conn_01x04_Pin" (at 42.545 142.24 0)
+    (property "Value" "Temp Sensor" (at 42.545 142.24 0)
       (effects (font (size 1.27 1.27)))
     )
@@
       (effects (font (size 1.27 1.27)) hide)
     )
-    (property "Datasheet" "~" (at 41.91 147.32 0)
+    (property "Datasheet" "https://tools.molex.com/pdm_docs/sd/436500400_sd.pdf" (at 41.91 147.32 0)
       (effects (font (size 1.27 1.27)) hide)
     )
@@
       (effects (font (size 1.27 1.27)) hide)
     )
-    (property "Datasheet" "~" (at 88.9 146.05 0)
+    (property "Datasheet" "https://www.yageo.com/upload/media/product/app/datasheet/rchip/pyu-rt_1-to-0.01_rohs_l.pdf" (at 88.9 146.05 0)
       (effects (font (size 1.27 1.27)) hide)
     )
@@
       (effects (font (size 1.27 1.27)) hide)
     )
-    (property "Catalog No" "YAG2302CT-ND" (at 88.9 146.05 0)
-      (effects (font (size 1.27 1.27)) hide)
-    )
+    (property "Catalog No" "13-RT1206FRE0715KLCT-ND" (at 88.9 146.05 0)
+      (effects (font (size 1.27 1.27)) hide)
+    )

Commit message: fixes
Parts:
- added R7, R8: 4.7 kΩ, Resistor_SMD:R_1206_3216Metric_Pad1.30x1.75mm_HandSolder, symbol Device:R_US
- A1: Catalog No (none) -> 1050-ABX00033-ND; Vendor (none) -> Digikey
- R1, R2, R3, R4, R5, R6: Indicator + -> (none)
Connections:
- net +5V: now also A1.5V, R7.1, R8.1
- net A4: now also R8.2
- net A5: now also R7.2
- net GND: now also A1.GND1 (GND)
- net +3V3: now reaches A1.3V3 (3.3V)
Other:
- moved on the sheet: J3

Commit message: updated bom
Parts:
- U1: Catalog No 296-13869-5-ND -> https://www.ti.com/lit/ds/symlink/lm117.pdf?HQS=dis-dk-null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
Changed lines of the file:
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@@
       (effects (font (size 1.27 1.27)) hide)
     )
-    (property "Catalog No" "296-13869-5-ND" (at 92.71 38.1 0)
+    (property "Catalog No" "https://www.ti.com/lit/ds/symlink/lm117.pdf?HQS=dis-dk-null-digikeymode-dsf-pf-null-wwe&ts=1708276608887&ref_url=https%253A%252F%252Fwww.ti.com%252Fgeneral%252Fdocs%252Fsuppproductinfo.tsp%253FdistId%253D10%2526gotoUrl%253Dhttps%253A%252F%252Fwww.ti.com%252Flit%252Fgpn%252Flm117" (at 92.71 38.1 0)
       (effects (font (size 1.27 1.27)) hide)
     )
