File: kicad/V2/heaterboard-2.kicad_pcb (KiCad board)
At the start: 4 copper layers, 113.2 x 68.2 mm, 15 parts, among them J1 Screw_Terminal_01x02, J2 Screw_Terminal_01x02, J3 Conn_01x04_Pin, J4 Conn_01x05_Pin, Q1 Q_NMOS_GDS, U1 LM317_TO-220

Commit message: more update
Changed lines of the file:
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@@
     (property "ki_keywords" "R res resistor")
     (attr smd)
-    (fp_text reference "R2" (at 0 -1.82 90) (layer "F.SilkS")
+    (fp_text reference "R2" (at 3.53 0 180) (layer "F.SilkS")
         (effects (font (size 1 1) (thickness 0.15)))
     )
@@
     (property "ki_keywords" "R res resistor")
     (attr smd)
-    (fp_text reference "R6" (at 0 -1.82 90) (layer "F.SilkS")
+    (fp_text reference "R6" (at 3.53 0 180) (layer "F.SilkS")
         (effects (font (size 1 1) (thickness 0.15)))
     )
@@
     (property "Sheetfile" "heaterboard-2.kicad_sch")
     (property "Sheetname" "")
-    (property "ki_description" "Polarized capacitor, US symbol")
+    (property "ki_description" "Unpolarized capacitor")
     (property "ki_keywords" "cap capacitor")
     (attr smd)
-    (fp_text reference "C2" (at 0 -1.85 90) (layer "F.SilkS")
+    (fp_text reference "C2" (at 3.4675 0 180) (layer "F.SilkS")
         (effects (font (size 1 1) (thickness 0.15)))
     )
@@
     (property "ki_keywords" "R res resistor")
     (attr smd)
-    (fp_text reference "R4" (at 0 -1.82 90) (layer "F.SilkS")
+    (fp_text reference "R4" (at 3.53 0 180) (layer "F.SilkS")
         (effects (font (size 1 1) (thickness 0.15)))
     )
@@
     (property "ki_keywords" "R res resistor")
     (attr smd)
-    (fp_text reference "R1" (at 0 -1.82 90) (layer "F.SilkS")
+    (fp_text reference "R1" (at 3.455 0 180) (layer "F.SilkS")
         (effects (font (size 1 1) (thickness 0.15)))
     )
@@
     (property "ki_keywords" "R res resistor")
     (attr smd)
-    (fp_text reference "R5" (at 0 -1.82 90) (layer "F.SilkS")
+    (fp_text reference "R5" (at 3.53 0 180) (layer "F.SilkS")
         (effects (font (size 1 1) (thickness 0.15)))
     )
@@
     (property "ki_keywords" "R res resistor")
     (attr smd)
-    (fp_text reference "R3" (at 0 -1.82 90) (layer "F.SilkS")
+    (fp_text reference "R3" (at 3.53 0 180) (layer "F.SilkS")
         (effects (font (size 1 1) (thickness 0.15)))
     )
@@
     (property "ki_keywords" "connector")
     (attr through_hole)
-    (fp_text reference "J3" (at 4.5 -10.12 180) (layer "F.SilkS")
-        (effects (font (size 1 1) (thickness 0.15)))
-    )
-    (fp_text value "Conn_01x04_Pin" (at 4.5 3.22 180) (layer "F.Fab")
+    (fp_text reference "J3" (at 4.5 2.665 180) (layer "F.SilkS")
+        (effects (font (size 1 1) (thickness 0.15)))
+    )
+    (fp_text value "Conn_01x04_Pin" (at 4.5 -10.67 180) (layer "F.Fab")
         (effects (font (size 1 1) (thickness 0.15)))
     )
@@
     (property "ki_keywords" "cap capacitor")
     (attr smd)
-    (fp_text reference "C1" (at 0 -1.85 90) (layer "F.SilkS")
-        (effects (font (size 1 1) (thickness 0.15)))
-    )
+    (fp_text reference "C1" (at 3.4675 0 180) (layer "F.SilkS")
+        (effects (font (size 1 1) (thickness 0.15)))
+    )

Commit message: Routing, parts, bom
Parts:
- J1: value Screw_Terminal_01x02 -> Power In
- J2: value Screw_Terminal_01x02 -> Heater Connect
- J3: value Conn_01x04_Pin -> Temp Sensor
- J4: value Conn_01x05_Pin -> Relay
Connections:
- R3 pad 2: /A0 -> /A6
- R4 pad 1: /A0 -> /A6
- R5 pad 2: /A1 -> /A7
- R6 pad 1: /A1 -> /A7
Routing:
- net /A1: track 44.5 -> 0.00 mm
- net /A0: track 31.0 -> 0.00 mm
- net /A7: track 0.00 -> 29.0 mm
- net /A6: track 0.00 -> 17.3 mm
- net +9V: track 75.6 -> 72.7 mm, vias 0 -> 2
Other:
- board text added: "12V IN"
- board text added: "BOSTON UNIVERSITY ENG-ME-692 WINDSHIELD HEATER PROJECT AL LEVINE & ZEWEI WU"
- board text added: "HEATER"
- board text added: "RELAY"
- board text added: "TEMP SENSOR"

Commit message: fixes
Parts:
- added R7: 4.7 kΩ, Resistor_SMD:R_1206_3216Metric_Pad1.30x1.75mm_HandSolder, F.Cu at (156.8, 89.9)
- added R8: 4.7 kΩ, Resistor_SMD:R_1206_3216Metric_Pad1.30x1.75mm_HandSolder, F.Cu at (153.0, 89.9)
- moved J4 1.91 mm to (154.9, 79.4)
Connections:
- A1 pad 3V3: unconnected-(A1-3.3V-Pad3V3) -> +3V3
- A1 pad 5V: unconnected-(A1-Pad5V) -> +5V
- A1 pad GND1: unconnected-(A1-GND-PadGND1) -> GND
Routing:
- net +5V: track 0.00 -> 47.6 mm, vias 0 -> 4
- net Net-(J4-Pin_3): track 10.9 -> 9.01 mm
- net +12V: track 3.86 -> 4.65 mm
Other:
- board text added: "ARDUINO"
- board text added: "USB"
