File: kicad/V2/heaterboard-2.kicad_pcb (KiCad board)
At the start: 4 copper layers, 113.2 x 68.2 mm, 17 parts, among them J1 Power In, J2 Heater Connect, J3 Temp Sensor, J4 Relay, Q1 Q_NMOS_GDS, U1 LM317_TO-220

Commit message: gerbers fix
Other:
- board text added: "JLCJLCJLCJLC"
Changed lines of the file:
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@@
     (effects (font (size 1 1) (thickness 0.2) bold) (justify left top))
+  )
+  (gr_text "JLCJLCJLCJLC" (at 80.01 121.92) (layer "F.SilkS")
+    (effects (font (size 1 1) (thickness 0.15)) (justify left bottom))
   )
   (segment (start 153.035 90.805) (end 151.13 88.9) (width 0.25) (layer "F.Cu") (net 6))
