File: kicad/V3/heaterboard-3/heaterboard-3.kicad_pcb (KiCad board)
At the start: 4 copper layers, 113.2 x 68.2 mm, 17 parts, among them J1 Power In, J2 Heater Connect, J3 Temp Sensor, J4 Relay, Q1 Q_NMOS_GDS, U1 LM317_TO-220

Commit message: board r3 update
Parts:
- removed J3: Temp Sensor, Connector_Molex:Molex_Micro-Fit_3.0_43650-0400_1x04_P3.00mm_Horizontal
- added C3: 0.1μF, Capacitor_SMD:C_1206_3216Metric_Pad1.33x1.80mm_HandSolder, F.Cu at (102.9, 67.6)
- added C4: 0.1μF, Capacitor_SMD:C_1206_3216Metric_Pad1.33x1.80mm_HandSolder, F.Cu at (118.1, 67.6)
- added J5: GPIO Headers, Connector_PinSocket_2.54mm:PinSocket_1x15_P2.54mm_Vertical, F.Cu at (124.5, 63.5)
- added J6: GPIO Headers, Connector_PinSocket_2.54mm:PinSocket_1x15_P2.54mm_Vertical, F.Cu at (149.9, 63.5)
- added R10: 3.32kΩ, Resistor_SMD:R_1206_3216Metric_Pad1.30x1.75mm_HandSolder, F.Cu at (114.3, 67.6)
- added R9: 6.65kΩ, Resistor_SMD:R_1206_3216Metric_Pad1.30x1.75mm_HandSolder, F.Cu at (110.5, 67.6)
- added U2: Current Sensor IC, Package_SO:SOIC-8_3.9x4.9mm_P1.27mm, F.Cu at (97.2, 101.6)
- A1: value Arduino_Nano_Socket -> Arduino Nano
- C1: value 100nF -> 0.1μF
- J2: value Heater Connect -> Heater; footprint Connector_Molex:Molex_Mega-Fit_76825-0002_2x01_P5.70mm_Horizontal -> Connector_Molex:Molex_Mega-Fit_76825-0004_2x02_P5.70mm_Horizontal
- Q1: value Q_NMOS_GDS -> Power MOSFET
- R1: value 0.4kΩ -> 1kΩ
- R2: value 2.4kΩ -> 3kΩ
- R3: value 10 kΩ -> 10kΩ
- R4, R6: value 5 kΩ -> 5kΩ
- R5: value 15 kΩ -> 15kΩ
- R7: value 4.7 kΩ -> 6.65kΩ
- R8: value 4.7 kΩ -> 3.32kΩ
- U1: value LM317_TO-220 -> Voltage Regulator
- moved R7 61.9 mm to (99.1, 67.6), turned to 90 degrees
- moved R8 51.4 mm to (106.7, 67.6)
- moved R1 11.9 mm to (83.8, 67.7)
- moved R2 11.9 mm to (87.6, 67.7)
- moved C1 11.9 mm to (95.2, 67.7)
- moved C2 11.9 mm to (91.4, 67.7)
- moved Q1 11.1 mm to (94.6, 88.9)
- moved R3 7.11 mm to (160.0, 67.6)
- moved R4 7.11 mm to (163.8, 67.6), turned to -90 degrees
- moved R5 7.11 mm to (167.6, 67.6)
- moved R6 7.11 mm to (171.4, 67.6), turned to -90 degrees
- moved U1 6.70 mm to (94.6, 76.8)
- moved J4 3.74 mm to (156.9, 76.2)
- moved J2 2.85 mm to (114.9, 88.9)
- moved J1 2.14 mm to (85.1, 88.9)
Connections:
- A1 pad RST1: unconnected-(A1-RESET-PadRST1) -> /RST1
- A1 pad RST2: unconnected-(A1-RESET-PadRST2) -> /RST2
- A1 pad VIN: +9V -> +5V
- C2 pad 1: +9V -> +5V
- J2 pad 2: +12V -> Net-(J2-Pin_2)
- Q1 pad 2: Net-(J2-Pin_1) -> Net-(J2-Pin_2)
- R1 pad 1: +9V -> +5V
- R7 pad 1: +5V -> Net-(J2-Pin_4)
- R7 pad 2: /A5 -> /A0
- R8 pad 1: +5V -> /A0
- R8 pad 2: /A4 -> GND
- U1 pad 2: +9V -> +5V
Routing:
- net /A0: track 0.00 -> 93.1 mm
- net +5V: track 47.6 -> 128.1 mm, vias 4 -> 3
- net +9V: track 72.7 -> 0.00 mm, vias 2 -> 0
- net /A1: track 0.00 -> 71.0 mm
- net /D9: track 33.6 -> 5.08 mm
- net Net-(J2-Pin_1): track 0.00 -> 24.2 mm
- net Net-(J2-Pin_4): track 0.00 -> 20.7 mm
- net /A5: track 22.1 -> 5.08 mm
- net Net-(J2-Pin_3): track 0.00 -> 16.1 mm
- net Net-(J2-Pin_2): track 0.00 -> 13.6 mm
- net /A4: track 17.9 -> 5.08 mm
- net GND: track 9.75 -> 17.9 mm, vias 5 -> 10
- net /A6: track 17.3 -> 24.7 mm
- net +12V: track 4.65 -> 10.9 mm, vias 2 -> 4
- net /A7: track 29.0 -> 34.3 mm
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Other:
- board text added: "BOSTON UNIVERSITY ENG-ME-692 WINDSHIELD HEATER PROJECT REV. 3 AL LEVINE & ZEWEI WU"
- board text removed: "12V IN"
- board text removed: "ARDUINO"
- board text removed: "BOSTON UNIVERSITY ENG-ME-692 WINDSHIELD HEATER PROJECT AL LEVINE & ZEWEI WU"
- board text removed: "HEATER"
- board text removed: "RELAY"
- board text removed: "TEMP SENSOR"
