File: kicad/V3/heaterboard-3/heaterboard-3.kicad_sch (KiCad schematic)
At the start: 17 parts, among them J1 Power In, J2 Heater Connect, J3 Temp Sensor, J4 Relay, Q1 Q_NMOS_GDS, U1 LM317_TO-220

Commit message: board r3 update
Parts:
- removed J2: Heater Connect, Connector_Molex:Molex_Mega-Fit_76825-0002_2x01_P5.70mm_Horizontal, symbol Connector:Screw_Terminal_01x02
- removed J3: Temp Sensor, Connector_Molex:Molex_Micro-Fit_3.0_43650-0400_1x04_P3.00mm_Horizontal, symbol Connector:Conn_01x04_Pin
- added C3, C4: 0.1μF, Capacitor_SMD:C_1206_3216Metric_Pad1.33x1.80mm_HandSolder, symbol Device:C
- added J2: Heater, Connector_Molex:Molex_Mega-Fit_76825-0004_2x02_P5.70mm_Horizontal, symbol Connector:Conn_01x04_Pin
- added J5, J6: GPIO Headers, Connector_PinSocket_2.54mm:PinSocket_1x15_P2.54mm_Vertical, symbol Connector:Screw_Terminal_01x15
- added R10: 3.32kΩ, Resistor_SMD:R_1206_3216Metric_Pad1.30x1.75mm_HandSolder, symbol Device:R_US
- added R9: 6.65kΩ, Resistor_SMD:R_1206_3216Metric_Pad1.30x1.75mm_HandSolder, symbol Device:R_US
- added U2: Current Sensor IC, Package_SO:SOIC-8_3.9x4.9mm_P1.27mm, symbol Sensor_Current:ACS712xLCTR-20A
- A1: value Arduino_Nano_Socket -> Arduino Nano
- C1: value 100nF -> 0.1μF
- Q1: value Q_NMOS_GDS -> Power MOSFET
- R1: value 0.4kΩ -> 1kΩ
- R2: value 2.4kΩ -> 3kΩ
- R3: value 10 kΩ -> 10kΩ
- R4, R6: value 5 kΩ -> 5kΩ
- R5: value 15 kΩ -> 15kΩ
- R7: value 4.7 kΩ -> 6.65kΩ; Catalog No YAG3966CT-ND -> 311-6.65KFRCT-ND
- R8: value 4.7 kΩ -> 3.32kΩ; Catalog No YAG3966CT-ND -> 311-3.32KFRCT-ND
- U1: value LM317_TO-220 -> Voltage Regulator; Catalog No https://www.ti.com/lit/ds/symlink/lm117.pdf?HQS=dis-dk-null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 -> LM317TNS/NOPB-ND
Connections:
- net +9V is gone; now on net +5V: A1.VIN, C2.1, R1.1, U1.2 (VO)
- net +12V: now also U2.1 (IP+), U2.2 (IP+)
- net +3V3: now also J6.14 (Pin_14)
- net +5V: now also J6.1 (Pin_1), J6.4 (Pin_4), U2.8 (VCC); no longer R7.1, R8.1
- net A0: now also R7.2, R8.1, C3.1, J6.12 (Pin_12)
- net A1: now also C4.1, J6.11 (Pin_11), R10.1, R9.2
- net A2: now also J6.10 (Pin_10), U2.7 (VIOUT)
- net A3: now also J6.9 (Pin_9)
- net A4: now also J6.8 (Pin_8); no longer R8.2
- net A5: now also J6.7 (Pin_7); no longer R7.2
- net A6: now also J6.6 (Pin_6)
- net A7: now also J6.5 (Pin_5)
- net AREF: now also J6.13 (Pin_13)
- net D0: now also J5.2 (Pin_2)
- net D1: now also J5.1 (Pin_1)
- net D10: now also J5.13 (Pin_13)
- net D11: now also J5.14 (Pin_14)
- net D12: now also J5.15 (Pin_15)
- net D13: now also J6.15 (Pin_15)
- net D2: now also J5.5 (Pin_5)
- net D3: now also J5.6 (Pin_6)
- net D4: now also J5.7 (Pin_7)
- net D5: now also J5.8 (Pin_8)
- net D6: now also J5.9 (Pin_9)
- net D7: now also J5.10 (Pin_10)
- net D8: now also J5.11 (Pin_11)
- net D9: now also J5.12 (Pin_12)
- net GND: now also R8.2, C3.2, C4.2, J5.4 (Pin_4), J6.2 (Pin_2), R10.2, U2.5 (GND)
- net at Q1.2 (D): now also J2.2 (Pin_2)
- net RST1: now reaches A1.RST1 (RESET)
- net RST1: now also J5.3 (Pin_3)
- net RST2: now reaches A1.RST2 (RESET)
- net RST2: now also J6.3 (Pin_3)
- new net: J2.1 (Pin_1), U2.3 (IP-), U2.4 (IP-)
- new net: J2.3 (Pin_3), R9.1
- new net: J2.4 (Pin_4), R7.1
Other:
- note added: "GPIO HEADERS"
- note added: "HEATER POWER CONTROL & REMOTE SENSING"
- note removed: "HEATER POWER CONTROL"
- note removed: "TEMPERATURE MODULE"
- moved on the sheet: A1, J1, J4, Q1, R3, R4, R5, R6
